Commit message: Add files via upload

File: simulation_ws/src/jetbot_description/urdf/jetbot.urdf (robot description, URDF)
Before this commit: robot JetBot, 4 links, 3 joints
Links:
- added link base_link
Joints:
- added joint base_link_to_chassis: type fixed, parent base_link, child JetBot__chassis
- joint JetBot__left_wheel_hinge: parent JetBot__chassis -> base_link
- joint JetBot__right_wheel_hinge: parent JetBot__chassis -> base_link

Commit message: Revised the transform tree

File: simulation_ws/src/jetbot_description/urdf/jetbot.urdf (robot description, URDF)
Before this commit: robot JetBot, 5 links, 4 joints
Links:
- added link JetBot__lidar_link, mass 0.01; visual box size=0.001 0.001 0.001
Joints:
- added joint JetBot__lidar_joint: type fixed, parent JetBot__chassis, child JetBot__lidar_link, origin xyz=0.055   0      0.1857 rpy=0    0  0, axis 0.96891  0       0.2474
- joint JetBot__left_wheel_hinge: parent base_link -> JetBot__chassis
- joint JetBot__right_wheel_hinge: parent base_link -> JetBot__chassis
