Commit message: ani

File: simulation_ws/src/jetbot_description/models/urdf/jetbot.urdf (robot description, URDF)
Before this commit: robot JetBot, 6 links, 5 joints
Links:
- link JetBot__chassis: geometry collision mesh filename=package://meshes/JetBot-v3-Chassis.dae scale=0.001 0.001 0.001; visual mesh filename=package://meshes/JetBot-v3-Chassis.dae scale=0.001 0.001 0.001
- link JetBot__left_wheel: geometry collision cylinder length=0.008 radius=0.030; visual mesh filename=package://meshes/JetBot-v3-Wheel.stl scale=0.001 0.001 0.001
- link JetBot__right_wheel: geometry collision cylinder length=0.008 radius=0.030; visual mesh filename=package://meshes/JetBot-v3-Wheel.stl scale=0.001 0.001 0.001

Commit message: ani

File: simulation_ws/src/jetbot_description/models/urdf/jetbot.urdf (robot description, URDF)
Before this commit: robot JetBot, 6 links, 5 joints
Links:
- removed link base_footprint
- removed link camera_link
- removed link left_wheel
- removed link lidar_link
- removed link right_wheel
- added link JetBot__camera_link, mass 0.01; visual box size=0.001 0.001 0.001
- added link JetBot__chassis, mass 1.0; collision mesh filename=package://meshes/JetBot-v3-Chassis.dae scale=0.001 0.001 0.001; visual mesh filename=package://meshes/JetBot-v3-Chassis.dae scale=0.001 0.001 0.001
- added link JetBot__left_wheel, mass 0.1; collision cylinder length=0.008 radius=0.030; visual mesh filename=package://meshes/JetBot-v3-Wheel.stl scale=0.001 0.001 0.001
- added link JetBot__lidar_link, mass 0.01; visual box size=0.001 0.001 0.001
- added link JetBot__right_wheel, mass 0.1; collision cylinder length=0.008 radius=0.030; visual mesh filename=package://meshes/JetBot-v3-Wheel.stl scale=0.001 0.001 0.001
- link base_link: mass 1.0 -> None; geometry 
Joints:
- removed joint base_joint
- removed joint camera_joint
- removed joint left_wheel_hinge
- removed joint lidar_joint
- removed joint right_wheel_hinge
- added joint JetBot__camera_joint: type fixed, parent JetBot__chassis, child JetBot__camera_link, origin xyz=0.055   0      0.0857 rpy=0    0.25  0, axis 0.96891  0       0.2474
- added joint JetBot__left_wheel_hinge: type continuous, parent JetBot__chassis, child JetBot__left_wheel, origin xyz=0.03     0.05125  0.03 rpy=0       0       1.57079, axis 1  0  0
- added joint JetBot__lidar_joint: type fixed, parent JetBot__chassis, child JetBot__lidar_link, origin xyz=0.055   0      0.1857 rpy=0    0  0, axis 0.96891  0       0.2474
- added joint JetBot__right_wheel_hinge: type continuous, parent JetBot__chassis, child JetBot__right_wheel, origin xyz=0.03   -0.0595  0.03 rpy=0       0       1.57079, axis 1  0  0
- added joint base_link_to_chassis: type fixed, parent base_link, child JetBot__chassis
